Commit message: Updates to rdf linked ultrasonic sensor to model

File: picarx/script/picarx.urdf.xacro (robot description, xacro)
@@ -2,20 +2,46 @@
 <robot xmlns:xacro="http://www.ros.org/wiki/xacro" name="picarx_bot">
     <!-- Properties -->
-    <xacro:property name="body_length" value="1.91" />
-    <xacro:property name="body_width" value="0.680618" />
-    <xacro:property name="body_height" value="1.065022" />
+    <xacro:property name="body_length" value=".22" />
+    <xacro:property name="body_width" value="0.085" />
+    <xacro:property name="body_height" value="0.04" />
     <xacro:property name="body_mass" value="20.3" />
-    <xacro:property name="front_wheel_width" value=".254" />
-    <xacro:property name="front_wheel_diameter" value="0.605" />
-    <xacro:property name="rear_wheel_width" value=".3175" />
-    <xacro:property name="rear_wheel_diameter" value="0.635" />
+    <xacro:property name="front_wheel_width" value=".025" />
+    <xacro:property name="front_wheel_diameter" value="0.065" />
+    <xacro:property name="rear_wheel_width" value=".025" />
+    <xacro:property name="rear_wheel_diameter" value="0.065" />
+    <xacro:property name="base_link_z" value="${rear_wheel_diameter/2}" />
+    <!-- Materials -->
+    <material name="Blue">
+        <color rgba="0 0 1 1" />
+    </material>
+    <material name="Red">
+        <color rgba="1 0 0 1" />
+    </material>
+    <material name="Green">
+        <color rgba="0 1 0 1" />
+    </material>
+    <material name="Yellow">
+        <color rgba="1 1 0 1" />
+    </material>
+    <material name="Gray">
+        <color rgba="0.5 0.5 0.5 1" />
+    </material>
+    <material name="Black">
+        <color rgba="0 0 0 1" />
+    </material>
+    <material name="Orange">
+        <color rgba="1 0.5 0 1" />
+    </material>
     <!-- Base Link -->
     <link name="base_link">
         <visual>
+            <origin xyz="0 0 ${base_link_z + body_height/2}" rpy="0 0 0" />
             <geometry>
                 <box size="${body_length} ${body_width} ${body_height}" />
             </geometry>
-        </visual>
-        <collision>
+            <material name="Orange" />
+        </visual>
+        <collision>
+            <origin xyz="0 0 ${base_link_z + body_height/2}" rpy="0 0 0" />
             <geometry>
                 <box size="${body_length} ${body_width} ${body_height}" />
@@ -23,54 +49,118 @@
         </collision>
     </link>
-    <!-- Steering Joints -->
-    <link name="left_steer">
-        <visual>
-            <geometry>
-                <cylinder length="0.05" radius="0.03" />
-            </geometry>
-            <material name="Blue">
-                <color rgba="0 0 1 1" />
-            </material>
-        </visual>
-    </link>
-    <link name="right_steer">
-        <visual>
-            <geometry>
-                <cylinder length="0.05" radius="0.03" />
-            </geometry>
-            <material name="Red">
-                <color rgba="1 0 0 1" />
-            </material>
-        </visual>
-    </link>
-    <joint name="left_steer_joint" type="revolute">
+    <!-- Steering Link (Ackermann) -->
+    <link name="steering_link">
+        <visual>
+            <origin xyz="0 0 0" rpy="0 0 0" />
+            <geometry>
+                <box size="0.02 0.07 0.01" />
+            </geometry>
+            <material name="Gray" />
+        </visual>
+        <collision>
+            <origin xyz="0 0 0" rpy="0 0 0" />
+            <geometry>
+                <box size="0.02 0.07 0.01" />
+            </geometry>
+        </collision>
+        <inertial>
+            <origin xyz="0 0 0" rpy="0 0 0" />
+            <mass value="0.2" />
+            <inertia ixx="0.0002" ixy="0" ixz="0" iyy="0.0002" iyz="0" izz="0.0002" />
+        </inertial>
+    </link>
+    <joint name="steering_joint" type="revolute">
         <parent link="base_link" />
-        <child link="left_steer" />
+        <child link="steering_link" />
+        <origin xyz="0.035 0 ${base_link_z}" rpy="0 0 0" />
         <axis xyz="0 0 1" />
-        <origin xyz="0.7 0.1 0.0" rpy="0 0 0" />
-        <limit lower="-0.50" upper="0.50" effort="1" velocity="3" />
-    </joint>
-    <joint name="right_steer_joint" type="revolute">
-        <parent link="base_link" />
-        <child link="right_steer" />
-        <axis xyz="0 0 1" />
-        <origin xyz="0.7 -0.1 0.0" rpy="0 0 0" />
-        <limit lower="-0.50" upper="0.50" effort="1" velocity="3" />
-    </joint>
-    <!-- Rear Wheels -->
+        <limit lower="-0.5" upper="0.5" effort="1" velocity="3" />
+    </joint>
+    <!-- Additional Steering Joints for Compatibility -->
+    <link name="left_steering_link"/>
+    <link name="right_steering_link"/>
+    <joint name="left_steering_joint" type="revolute">
+        <parent link="steering_link"/>
+        <child link="left_steering_link"/>
+        <origin xyz="0 0.03 0" rpy="0 0 0"/>
+        <axis xyz="0 0 1"/>
+        <limit lower="0.0" upper="0.0" effort="1" velocity="1"/>
+    </joint>
+    <joint name="right_steering_joint" type="revolute">
+        <parent link="steering_link"/>
+        <child link="right_steering_link"/>
+        <origin xyz="0 -0.03 0" rpy="0 0 0"/>
+        <axis xyz="0 0 1"/>
+        <limit lower="0.0" upper="0.0" effort="1" velocity="1"/>
+    </joint>
+    <!-- Front Wheels (fixed to steering link) -->
+    <link name="left_front_wheel">
+        <visual>
+            <origin xyz="0 0 0" rpy="1.5708 0 0" />
+            <geometry>
+                <cylinder length="${front_wheel_width}" radius="${front_wheel_diameter/2}" />
+            </geometry>
+            <material name="Green" />
+        </visual>
+        <collision>
+            <origin xyz="0 0 0" rpy="1.5708 0 0" />
+            <geometry>
+                <cylinder length="${front_wheel_width}" radius="${front_wheel_diameter/2}" />
+            </geometry>
+        </collision>
+        <inertial>
+            <origin xyz="0 0 0" rpy="0 0 0" />
+            <mass value="0.2" />
+            <inertia ixx="0.0002" ixy="0" ixz="0" iyy="0.0002" iyz="0" izz="0.0002" />
+        </inertial>
+    </link>
+    <link name="right_front_wheel">
+        <visual>
+            <origin xyz="0 0 0" rpy="1.5708 0 0" />
+            <geometry>
+                <cylinder length="${front_wheel_width}" radius="${front_wheel_diameter/2}" />
+            </geometry>
+            <material name="Red" />
+        </visual>
+        <collision>
+            <origin xyz="0 0 0" rpy="1.5708 0 0" />
+            <geometry>
+                <cylinder length="${front_wheel_width}" radius="${front_wheel_diameter/2}" />
+            </geometry>
+        </collision>
+        <inertial>
+            <origin xyz="0 0 0" rpy="0 0 0" />
+            <mass value="0.2" />
+            <inertia ixx="0.0002" ixy="0" ixz="0" iyy="0.0002" iyz="0" izz="0.0002" />
+        </inertial>
+    </link>
+    <joint name="left_front_wheel_joint" type="fixed">
+        <parent link="left_steering_link" />
+        <child link="left_front_wheel" />
+        <origin xyz="0 0.015 0" rpy="0 0 0" />
+    </joint>
+    <joint name="right_front_wheel_joint" type="fixed">
+        <parent link="right_steering_link" />
+        <child link="right_front_wheel" />
+        <origin xyz="0 -0.015 0" rpy="0 0 0" />
+    </joint>
+    <!-- Rear Wheels (driven, continuous) -->
     <link name="left_rear_wheel">
         <visual>
-            <geometry>
-                <cylinder length="${rear_wheel_width}" radius="${rear_wheel_diameter/2}" />
-            </geometry>
-        </visual>
-        <collision>
-            <geometry>
-                <cylinder length="${rear_wheel_width}" radius="${rear_wheel_diameter/2}" />
-            </geometry>
-        </collision>
-        <inertial>
+            <origin xyz="0 0 0" rpy="1.5708 0 0" />
+            <geometry>
+                <cylinder length="${rear_wheel_width}" radius="${rear_wheel_diameter/2}" />
+            </geometry>
+            <material name="Yellow" />
+        </visual>
+        <collision>
+            <origin xyz="0 0 0" rpy="1.5708 0 0" />
+            <geometry>
+                <cylinder length="${rear_wheel_width}" radius="${rear_wheel_diameter/2}" />
+            </geometry>
+        </collision>
+        <inertial>
+            <origin xyz="0 0 0" rpy="0 0 0" />
             <mass value="0.5" />
-            <origin xyz="0 0 0" />
             <inertia ixx="0.001" ixy="0" ixz="0" iyy="0.001" iyz="0" izz="0.001" />
         </inertial>
@@ -78,16 +168,19 @@
     <link name="right_rear_wheel">
         <visual>
-            <geometry>
-                <cylinder length="${rear_wheel_width}" radius="${rear_wheel_diameter/2}" />
-            </geometry>
-        </visual>
-        <collision>
-            <geometry>
-                <cylinder length="${rear_wheel_width}" radius="${rear_wheel_diameter/2}" />
-            </geometry>
-        </collision>
-        <inertial>
+            <origin xyz="0 0 0" rpy="1.5708 0 0" />
+            <geometry>
+                <cylinder length="${rear_wheel_width}" radius="${rear_wheel_diameter/2}" />
+            </geometry>
+            <material name="Yellow" />
+        </visual>
+        <collision>
+            <origin xyz="0 0 0" rpy="1.5708 0 0" />
+            <geometry>
+                <cylinder length="${rear_wheel_width}" radius="${rear_wheel_diameter/2}" />
+            </geometry>
+        </collision>
+        <inertial>
+            <origin xyz="0 0 0" rpy="0 0 0" />
             <mass value="0.5" />
-            <origin xyz="0 0 0" />
             <inertia ixx="0.001" ixy="0" ixz="0" iyy="0.001" iyz="0" izz="0.001" />
         </inertial>
@@ -96,54 +189,39 @@
         <parent link="base_link" />
         <child link="left_rear_wheel" />
-        <axis xyz="0.0 0.1 0.0" />
-        <origin xyz="-0.855 0.390309 0.0" />
+        <origin xyz="-0.065 0.045 ${base_link_z}" rpy="0 0 0" />
+        <axis xyz="0 1 0" />
     </joint>
     <joint name="right_rear_axle" type="continuous">
         <parent link="base_link" />
         <child link="right_rear_wheel" />
-        <axis xyz="0.0 0.1 0.0" />
-        <origin xyz="-0.855 -0.390309 0.0" />
-    </joint>
-    <!-- Transmissions -->
-    <transmission name="left_steer_joint_trans">
-        <type>transmission_interface/SimpleTransmission</type>
-        <joint name="left_steer_joint">
-            <hardwareInterface>hardware_interface/PositionJointInterface</hardwareInterface>
-        </joint>
-        <actuator name="left_steer_joint_motor">
-            <hardwareInterface>hardware_interface/PositionJointInterface</hardwareInterface>
-            <mechanicalReduction>1</mechanicalReduction>
-        </actuator>
-    </transmission>
-    <transmission name="right_steer_joint_trans">
-        <type>transmission_interface/SimpleTransmission</type>
-        <joint name="right_steer_joint">
-            <hardwareInterface>hardware_interface/PositionJointInterface</hardwareInterface>
-        </joint>
-        <actuator name="right_steer_joint_motor">
-            <hardwareInterface>hardware_interface/PositionJointInterface</hardwareInterface>
-            <mechanicalReduction>1</mechanicalReduction>
-        </actuator>
-    </transmission>
-    <transmission name="left_rear_wheel_joint_trans">
-        <type>transmission_interface/SimpleTransmission</type>
-        <joint name="left_rear_axle">
-            <hardwareInterface>hardware_interface/VelocityJointInterface</hardwareInterface>
-        </joint>
-        <actuator name="left_rear_wheel_motor">
-            <hardwareInterface>hardware_interface/VelocityJointInterface</hardwareInterface>
-            <mechanicalReduction>1</mechanicalReduction>
-        </actuator>
-    </transmission>
-    <transmission name="right_rear_wheel_joint_trans">
-        <type>transmission_interface/SimpleTransmission</type>
-        <joint name="right_rear_axle">
-            <hardwareInterface>hardware_interface/VelocityJointInterface</hardwareInterface>
-        </joint>
-        <actuator name="right_rear_wheel_motor">
-            <hardwareInterface>hardware_interface/VelocityJointInterface</hardwareInterface>
-            <mechanicalReduction>1</mechanicalReduction>
-        </actuator>
-    </transmission>
+        <origin xyz="-0.065 -0.045 ${base_link_z}" rpy="0 0 0" />
+        <axis xyz="0 1 0" />
+    </joint>
+    <!-- Ultrasonic Sensor -->
+    <link name="ultrasonic_link">
+        <visual>
+            <origin xyz="0.01 0 -${base_link_z-body_height/2}" rpy="0 1.5708 0"/>
+            <geometry>
+                <cylinder length="0.01" radius="0.01"/>
+            </geometry>
+            <material name="Blue"/>
+        </visual>
+        <collision>
+            <origin xyz="0 0 -${base_link_z-body_height/2}" rpy="0 0 0"/>
+            <geometry>
+                <cylinder length="0.01" radius="0.01"/>
+            </geometry>
+        </collision>
+        <inertial>
+            <origin xyz="0 0 0" rpy="0 0 0"/>
+            <mass value="0.01"/>
+            <inertia ixx="0.00001" ixy="0" ixz="0" iyy="0.00001" iyz="0" izz="0.00001"/>
+        </inertial>
+    </link>
+    <joint name="ultrasonic_joint" type="fixed">
+        <parent link="base_link"/>
+        <child link="ultrasonic_link"/>
+        <origin xyz="${body_length/2 - 0.005} 0 ${base_link_z + body_height}" rpy="0 0 0"/>
+    </joint>
     <!-- ros2_control block -->
     <ros2_control name="picarx_system" type="system">
@@ -153,5 +231,5 @@
             <param name="joint_states_topic">/topic_based_joint_states</param>
         </hardware>
-        <joint name="left_steer_joint">
+        <joint name="steering_joint">
             <command_interface name="position" />
             <state_interface name="position">
@@ -159,5 +237,5 @@
             </state_interface>
         </joint>
-        <joint name="right_steer_joint">
+        <joint name="left_steering_joint">
             <command_interface name="position" />
             <state_interface name="position">
@@ -165,8 +243,15 @@
             </state_interface>
         </joint>
+        <joint name="right_steering_joint">
+            <command_interface name="position" />
+            <state_interface name="position">
+                <param name="initial_value">0.0</param>
+            </state_interface>
+        </joint>
         <joint name="left_rear_axle">
             <state_interface name="velocity">
                 <param name="initial_value">0.0</param>
             </state_interface>
+            <state_interface name="position" />
             <command_interface name="velocity" />
         </joint>
@@ -175,4 +260,5 @@
                 <param name="initial_value">0.0</param>
             </state_interface>
+            <state_interface name="position" />
             <command_interface name="velocity" />
         </joint>

Commit message: More work on the urdf

File: picarx/script/picarx.urdf.xacro (robot description, xacro)
@@ -1,5 +1,6 @@
 <?xml version="1.0"?>
 <robot xmlns:xacro="http://www.ros.org/wiki/xacro" name="picarx_bot">
-    <!-- Properties -->
+    <!-- =================== Properties =================== -->
+    <!-- General properties of the robot -->
     <xacro:property name="body_length" value=".22" />
     <xacro:property name="body_width" value="0.085" />
@@ -11,5 +12,6 @@
     <xacro:property name="rear_wheel_diameter" value="0.065" />
     <xacro:property name="base_link_z" value="${rear_wheel_diameter/2}" />
-    <!-- Materials -->
+    <!-- =================== Materials ==================== -->
+    <!-- Define the materials used in the robot -->
     <material name="Blue">
         <color rgba="0 0 1 1" />
@@ -33,5 +35,6 @@
         <color rgba="1 0.5 0 1" />
     </material>
-    <!-- Base Link -->
+    <!-- =================== Base ========================= -->
+    <!-- Base link of the robot -->
     <link name="base_link">
         <visual>
@@ -49,5 +52,6 @@
         </collision>
     </link>
-    <!-- Steering Link (Ackermann) -->
+    <!-- =================== Steering ===================== -->
+    <!-- Steering mechanism of the robot -->
     <link name="steering_link">
         <visual>
@@ -78,20 +82,22 @@
     </joint>
     <!-- Additional Steering Joints for Compatibility -->
-    <link name="left_steering_link"/>
-    <link name="right_steering_link"/>
+    <link name="left_steering_link" />
+    <link name="right_steering_link" />
     <joint name="left_steering_joint" type="revolute">
-        <parent link="steering_link"/>
-        <child link="left_steering_link"/>
-        <origin xyz="0 0.03 0" rpy="0 0 0"/>
-        <axis xyz="0 0 1"/>
-        <limit lower="0.0" upper="0.0" effort="1" velocity="1"/>
+        <parent link="steering_link" />
+        <child link="left_steering_link" />
+        <origin xyz="0 0.03 0" rpy="0 0 0" />
+        <axis xyz="0 0 1" />
+        <limit lower="0.0" upper="0.0" effort="1" velocity="1" />
     </joint>
     <joint name="right_steering_joint" type="revolute">
-        <parent link="steering_link"/>
-        <child link="right_steering_link"/>
-        <origin xyz="0 -0.03 0" rpy="0 0 0"/>
-        <axis xyz="0 0 1"/>
-        <limit lower="0.0" upper="0.0" effort="1" velocity="1"/>
-    </joint>
+        <parent link="steering_link" />
+        <child link="right_steering_link" />
+        <origin xyz="0 -0.03 0" rpy="0 0 0" />
+        <axis xyz="0 0 1" />
+        <limit lower="0.0" upper="0.0" effort="1" velocity="1" />
+    </joint>
+    <!-- =================== Wheels ======================= -->
+    <!-- Define the wheels of the robot -->
     <!-- Front Wheels (fixed to steering link) -->
     <link name="left_front_wheel">
@@ -198,31 +204,116 @@
         <axis xyz="0 1 0" />
     </joint>
+    <!-- =================== Sensors ====================== -->
+    <!-- Define the sensors on the robot -->
     <!-- Ultrasonic Sensor -->
     <link name="ultrasonic_link">
         <visual>
-            <origin xyz="0.01 0 -${base_link_z-body_height/2}" rpy="0 1.5708 0"/>
-            <geometry>
-                <cylinder length="0.01" radius="0.01"/>
-            </geometry>
-            <material name="Blue"/>
-        </visual>
-        <collision>
-            <origin xyz="0 0 -${base_link_z-body_height/2}" rpy="0 0 0"/>
-            <geometry>
-                <cylinder length="0.01" radius="0.01"/>
-            </geometry>
-        </collision>
-        <inertial>
-            <origin xyz="0 0 0" rpy="0 0 0"/>
-            <mass value="0.01"/>
-            <inertia ixx="0.00001" ixy="0" ixz="0" iyy="0.00001" iyz="0" izz="0.00001"/>
+            <origin xyz="0.01 0 -${base_link_z-body_height/2}" rpy="0 1.5708 0" />
+            <geometry>
+                <cylinder length="0.01" radius="0.01" />
+            </geometry>
+            <material name="Blue" />
+        </visual>
+        <collision>
+            <origin xyz="0.01 0 -${base_link_z-body_height/2}" rpy="0 0 0" />
+            <geometry>
+                <cylinder length="0.01" radius="0.01" />
+            </geometry>
+        </collision>
+        <inertial>
+            <origin xyz="0 0 0" rpy="0 0 0" />
+            <mass value="0.01" />
+            <inertia ixx="0.00001" ixy="0" ixz="0" iyy="0.00001" iyz="0" izz="0.00001" />
         </inertial>
     </link>
     <joint name="ultrasonic_joint" type="fixed">
-        <parent link="base_link"/>
-        <child link="ultrasonic_link"/>
-        <origin xyz="${body_length/2 - 0.005} 0 ${base_link_z + body_height}" rpy="0 0 0"/>
-    </joint>
-    <!-- ros2_control block -->
+        <parent link="base_link" />
+        <child link="ultrasonic_link" />
+        <origin xyz="${body_length/2 - 0.005} 0 ${base_link_z + body_height}" rpy="0 0 0" />
+    </joint>
+    <!-- =================== Camera Pan-Tilt ============== -->
+    <!-- Define the camera and its pan-tilt mechanism -->
+    <link name="camera_pan_link">
+        <visual>
+            <origin xyz="0 0 0" rpy="0 0 0" />
+            <geometry>
+                <cylinder length="0.02" radius="0.015" />
+            </geometry>
+            <material name="Gray" />
+        </visual>
+        <collision>
+            <origin xyz="0 0 0" rpy="0 0 0" />
+            <geometry>
+                <cylinder length="0.02" radius="0.015" />
+            </geometry>
+        </collision>
+        <inertial>
+            <origin xyz="0 0 0" rpy="0 0 0" />
+            <mass value="0.02" />
+            <inertia ixx="0.00002" ixy="0" ixz="0" iyy="0.00002" iyz="0" izz="0.00002" />
+        </inertial>
+    </link>
+    <joint name="camera_pan_joint" type="revolute">
+        <parent link="base_link" />
+        <child link="camera_pan_link" />
+        <!-- Place the pan joint in front of the front wheels, at the same height as before -->
+        <origin xyz="${body_length/2 + 0.03} 0 ${base_link_z + body_height + 0.08}" rpy="0 0 0" />
+        <axis xyz="0 0 1" />
+        <limit lower="-1.5708" upper="1.5708" effort="1" velocity="1" />
+    </joint>
+    <link name="camera_tilt_link">
+        <visual>
+            <origin xyz="0 0 0" rpy="0 0 0" />
+            <geometry>
+                <cylinder length="0.02" radius="0.015" />
+            </geometry>
+            <material name="Gray" />
+        </visual>
+        <collision>
+            <origin xyz="0 0 0" rpy="0 0 0" />
+            <geometry>
+                <cylinder length="0.02" radius="0.015" />
+            </geometry>
+        </collision>
+        <inertial>
+            <origin xyz="0 0 0" rpy="0 0 0" />
+            <mass value="0.02" />
+            <inertia ixx="0.00002" ixy="0" ixz="0" iyy="0.00002" iyz="0" izz="0.00002" />
+        </inertial>
+    </link>
+    <joint name="camera_tilt_joint" type="revolute">
+        <parent link="camera_pan_link" />
+        <child link="camera_tilt_link" />
+        <origin xyz="0 0 0.02" rpy="0 0 0" />
+        <axis xyz="1 0 0" />
+        <limit lower="-1.5708" upper="1.5708" effort="1" velocity="1" />
+    </joint>
+    <link name="camera_link">
+        <visual>
+            <origin xyz="0 0 0" rpy="0 1.5708 0" />
+            <geometry>
+                <box size="0.03 0.03 0.03" />
+            </geometry>
+            <material name="Black" />
+        </visual>
+        <collision>
+            <origin xyz="0 0 0" rpy="0 1.5708 0" />
+            <geometry>
+                <box size="0.03 0.03 0.03" />
+            </geometry>
+        </collision>
+        <inertial>
+            <origin xyz="0 0 0" rpy="0 0 0" />
+            <mass value="0.05" />
+            <inertia ixx="0.00005" ixy="0" ixz="0" iyy="0.00005" iyz="0" izz="0.00005" />
+        </inertial>
+    </link>
+    <joint name="camera_link_joint" type="fixed">
+        <parent link="camera_tilt_link" />
+        <child link="camera_link" />
+        <origin xyz="0 0 0.02" rpy="0 0 0" />
+    </joint>
+    <!-- =================== ros2_control ================= -->
+    <!-- ros2_control configuration for the robot -->
     <ros2_control name="picarx_system" type="system">
         <hardware>
