Commit message: Fully implement the ackerman steering controller and topic based controller with Kilted

File: picarx/script/picarx.urdf.xacro (robot description, xacro)
@@ -36,6 +36,15 @@
     </material>
     <!-- =================== Base ========================= -->
+    <!-- Add odom link and fixed joint for TF root -->
+    <link name="odom" />
+    <joint name="odom_base_link" type="fixed">
+        <parent link="odom" />
+        <child link="base_link" />
+        <origin xyz="0 0 0" rpy="0 0 0" />
+    </joint>
     <!-- Base link of the robot -->
     <link name="base_link">
+    </link>
+    <link name="chassis_link">
         <visual>
             <origin xyz="0 0 ${base_link_z + body_height/2}" rpy="0 0 0" />
@@ -52,49 +61,52 @@
         </collision>
     </link>
+    <joint name="base_chassis_joint" type="fixed">
+        <parent link="base_link" />
+        <child link="chassis_link" />
+        <origin xyz="0 0 0" rpy="0 0 0 " />
+    </joint>
     <!-- =================== Steering ===================== -->
-    <!-- Steering mechanism of the robot -->
-    <link name="steering_link">
-        <visual>
-            <origin xyz="0 0 0" rpy="0 0 0" />
-            <geometry>
-                <box size="0.02 0.07 0.01" />
+    <!-- Additional Steering Joints for Compatibility -->
+    <link name="left_steering_link">
+        <visual>
+            <origin xyz="0 0 0" rpy="0 0 0" />
+            <geometry>
+                <cylinder length="0.01" radius="0.01" />
             </geometry>
             <material name="Gray" />
         </visual>
-        <collision>
-            <origin xyz="0 0 0" rpy="0 0 0" />
-            <geometry>
-                <box size="0.02 0.07 0.01" />
-            </geometry>
-        </collision>
-        <inertial>
-            <origin xyz="0 0 0" rpy="0 0 0" />
-            <mass value="0.2" />
-            <inertia ixx="0.0002" ixy="0" ixz="0" iyy="0.0002" iyz="0" izz="0.0002" />
-        </inertial>
-    </link>
-    <joint name="steering_joint" type="revolute">
-        <parent link="base_link" />
-        <child link="steering_link" />
-        <origin xyz="0.035 0 ${base_link_z}" rpy="0 0 0" />
+        <inertial>
+            <origin xyz="0 0 0" rpy="0 0 0" />
+            <mass value="0.01" />
+            <inertia ixx="0.00001" ixy="0" ixz="0" iyy="0.00001" iyz="0" izz="0.00001" />
+        </inertial>
+    </link>
+    <link name="right_steering_link">
+        <visual>
+            <origin xyz="0 0 0" rpy="0 0 0" />
+            <geometry>
+                <cylinder length="0.01" radius="0.01" />
+            </geometry>
+            <material name="Gray" />
+        </visual>
+        <inertial>
+            <origin xyz="0 0 0" rpy="0 0 0" />
+            <mass value="0.01" />
+            <inertia ixx="0.00001" ixy="0" ixz="0" iyy="0.00001" iyz="0" izz="0.00001" />
+        </inertial>
+    </link>
+    <joint name="left_steering_joint" type="revolute">
+        <parent link="base_link" />
+        <child link="left_steering_link" />
+        <origin xyz="0.035 0.03 ${base_link_z}" rpy="0 0 0" />
         <axis xyz="0 0 1" />
-        <limit lower="-0.5" upper="0.5" effort="1" velocity="3" />
-    </joint>
-    <!-- Additional Steering Joints for Compatibility -->
-    <link name="left_steering_link" />
-    <link name="right_steering_link" />
-    <joint name="left_steering_joint" type="revolute">
-        <parent link="steering_link" />
-        <child link="left_steering_link" />
-        <origin xyz="0 0.03 0" rpy="0 0 0" />
+        <limit lower="-0.56" upper="0.56" effort="10" velocity="7.5" />
+    </joint>
+    <joint name="right_steering_joint" type="revolute">
+        <parent link="base_link" />
+        <child link="right_steering_link" />
+        <origin xyz="0.035 -0.03 ${base_link_z}" rpy="0 0 0" />
         <axis xyz="0 0 1" />
-        <limit lower="0.0" upper="0.0" effort="1" velocity="1" />
-    </joint>
-    <joint name="right_steering_joint" type="revolute">
-        <parent link="steering_link" />
-        <child link="right_steering_link" />
-        <origin xyz="0 -0.03 0" rpy="0 0 0" />
-        <axis xyz="0 0 1" />
-        <limit lower="0.0" upper="0.0" effort="1" velocity="1" />
+        <limit lower="-0.56" upper="0.56" effort="10" velocity="7.5" />
     </joint>
     <!-- =================== Wheels ======================= -->
@@ -206,4 +218,30 @@
     <!-- =================== Sensors ====================== -->
     <!-- Define the sensors on the robot -->
+    <!-- IMU Sensor -->
+    <link name="imu_link">
+        <visual>
+            <origin xyz="0 0 ${base_link_z + body_height/2}" rpy="0 0 0" />
+            <geometry>
+                <box size="0.025 0.025 0.015" />
+            </geometry>
+            <material name="Blue" />
+        </visual>
+        <collision>
+            <origin xyz="0 0 ${base_link_z + body_height/2}" rpy="0 0 0" />
+            <geometry>
+                <box size="0.025 0.025 0.015" />
+            </geometry>
+        </collision>
+        <inertial>
+            <origin xyz="0 0 0" rpy="0 0 0" />
+            <mass value="0.01" />
+            <inertia ixx="0.00001" ixy="0" ixz="0" iyy="0.00001" iyz="0" izz="0.00001" />
+        </inertial>
+    </link>
+    <joint name="imu_joint" type="fixed">
+        <parent link="base_link" />
+        <child link="imu_link" />
+        <origin xyz="0 0 ${base_link_z + body_height/2}" rpy="0 0 0" />
+    </joint>
     <!-- Ultrasonic Sensor -->
     <link name="ultrasonic_link">
@@ -257,6 +295,5 @@
         <parent link="base_link" />
         <child link="camera_pan_link" />
-        <!-- Place the pan joint in front of the front wheels, at the same height as before -->
-        <origin xyz="${body_length/2 + 0.03} 0 ${base_link_z + body_height + 0.08}" rpy="0 0 0" />
+        <origin xyz="${body_length/2} 0 ${base_link_z + body_height}" rpy="0 0 0" />
         <axis xyz="0 0 1" />
         <limit lower="-1.5708" upper="1.5708" effort="1" velocity="1" />
@@ -286,5 +323,5 @@
         <child link="camera_tilt_link" />
         <origin xyz="0 0 0.02" rpy="0 0 0" />
-        <axis xyz="1 0 0" />
+        <axis xyz="0 -1 0" />
         <limit lower="-1.5708" upper="1.5708" effort="1" velocity="1" />
     </joint>
@@ -314,4 +351,7 @@
         <origin xyz="0 0 0.02" rpy="0 0 0" />
     </joint>
+    <!-- Static transforms for RViz2 visualization (for pan/tilt/camera) -->
+    <!-- Remove gazebo_ros_planar_move plugins, as they are not needed for RViz2 TF tree and may
+    cause confusion -->
     <!-- =================== ros2_control ================= -->
     <!-- ros2_control configuration for the robot -->
@@ -319,39 +359,145 @@
         <hardware>
             <plugin>topic_based_ros2_control/TopicBasedSystem</plugin>
-            <param name="joint_commands_topic">/topic_based_joint_commands</param>
-            <param name="joint_states_topic">/topic_based_joint_states</param>
         </hardware>
-        <joint name="steering_joint">
-            <command_interface name="position" />
-            <state_interface name="position">
-                <param name="initial_value">0.0</param>
-            </state_interface>
-        </joint>
         <joint name="left_steering_joint">
             <command_interface name="position" />
-            <state_interface name="position">
-                <param name="initial_value">0.0</param>
-            </state_interface>
+            <state_interface name="position" />
         </joint>
         <joint name="right_steering_joint">
             <command_interface name="position" />
-            <state_interface name="position">
-                <param name="initial_value">0.0</param>
-            </state_interface>
+            <state_interface name="position" />
         </joint>
         <joint name="left_rear_axle">
-            <state_interface name="velocity">
-                <param name="initial_value">0.0</param>
-            </state_interface>
+            <command_interface name="velocity" />
+            <state_interface name="velocity" />
             <state_interface name="position" />
+        </joint>
+        <joint name="right_rear_axle">
             <command_interface name="velocity" />
-        </joint>
+            <state_interface name="velocity" />
+            <state_interface name="position" />
+        </joint>
+    </ros2_control>
+    <!-- =================== Transmissions ================= -->
+    <!-- Required for ros2_control to map joints to actuators -->
+    <transmission name="left_steering_trans">
+        <type>transmission_interface/SimpleTransmission</type>
+        <joint name="left_steering_joint">
+            <hardwareInterface>position</hardwareInterface>
+        </joint>
+        <actuator name="left_steering_motor">
+            <hardwareInterface>position</hardwareInterface>
+            <mechanicalReduction>1</mechanicalReduction>
+        </actuator>
+    </transmission>
+    <transmission name="right_steering_trans">
+        <type>transmission_interface/SimpleTransmission</type>
+        <joint name="right_steering_joint">
+            <hardwareInterface>position</hardwareInterface>
+        </joint>
+        <actuator name="right_steering_motor">
+            <hardwareInterface>position</hardwareInterface>
+            <mechanicalReduction>1</mechanicalReduction>
+        </actuator>
+    </transmission>
+    <transmission name="left_rear_axle_trans">
+        <type>transmission_interface/SimpleTransmission</type>
+        <joint name="left_rear_axle">
+            <hardwareInterface>velocity</hardwareInterface>
+        </joint>
+        <actuator name="left_rear_motor">
+            <hardwareInterface>velocity</hardwareInterface>
+            <mechanicalReduction>1</mechanicalReduction>
+        </actuator>
+    </transmission>
+    <transmission name="right_rear_axle_trans">
+        <type>transmission_interface/SimpleTransmission</type>
         <joint name="right_rear_axle">
-            <state_interface name="velocity">
-                <param name="initial_value">0.0</param>
-            </state_interface>
-            <state_interface name="position" />
-            <command_interface name="velocity" />
-        </joint>
-    </ros2_control>
+            <hardwareInterface>velocity</hardwareInterface>
+        </joint>
+        <actuator name="right_rear_motor">
+            <hardwareInterface>velocity</hardwareInterface>
+            <mechanicalReduction>1</mechanicalReduction>
+        </actuator>
+    </transmission>
+    <!-- =================== Grayscale Sensors ============ -->
+    <!-- Three TCRT5000-based grayscale sensors at the front of the chassis, facing down -->
+    <link name="grayscale_0_link">
+        <visual>
+            <origin xyz="0 0 0" rpy="0 0 0" />
+            <geometry>
+                <cylinder length="0.01" radius="0.005" />
+            </geometry>
+            <material name="Black" />
+        </visual>
+        <collision>
+            <origin xyz="0 0 0" rpy="0 0 0" />
+            <geometry>
+                <cylinder length="0.01" radius="0.005" />
+            </geometry>
+        </collision>
+        <inertial>
+            <origin xyz="0 0 0" rpy="0 0 0" />
+            <mass value="0.001" />
+            <inertia ixx="0.000001" ixy="0" ixz="0" iyy="0.000001" iyz="0" izz="0.000001" />
+        </inertial>
+    </link>
+    <link name="grayscale_1_link">
+        <visual>
+            <origin xyz="0 0 0" rpy="0 0 0" />
+            <geometry>
+                <cylinder length="0.01" radius="0.005" />
+            </geometry>
+            <material name="Black" />
+        </visual>
+        <collision>
+            <origin xyz="0 0 0" rpy="0 0 0" />
+            <geometry>
+                <cylinder length="0.01" radius="0.005" />
+            </geometry>
+        </collision>
+        <inertial>
+            <origin xyz="0 0 0" rpy="0 0 0" />
+            <mass value="0.001" />
+            <inertia ixx="0.000001" ixy="0" ixz="0" iyy="0.000001" iyz="0" izz="0.000001" />
+        </inertial>
+    </link>
+    <link name="grayscale_2_link">
+        <visual>
+            <origin xyz="0 0 0" rpy="0 0 0" />
+            <geometry>
+                <cylinder length="0.01" radius="0.005" />
+            </geometry>
+            <material name="Black" />
+        </visual>
+        <collision>
+            <origin xyz="0 0 0" rpy="0 0 0" />
+            <geometry>
+                <cylinder length="0.01" radius="0.005" />
+            </geometry>
+        </collision>
+        <inertial>
+            <origin xyz="0 0 0" rpy="0 0 0" />
+            <mass value="0.001" />
+            <inertia ixx="0.000001" ixy="0" ixz="0" iyy="0.000001" iyz="0" izz="0.000001" />
+        </inertial>
+    </link>
+    <joint name="grayscale_0_joint" type="fixed">
+        <parent link="base_link" />
+        <!-- Slightly left, at the front, just below the chassis, facing down -->
+        <child link="grayscale_0_link" />
+        <origin xyz="${body_length/2} 0.015 ${base_link_z + 0.005}" rpy="0 1.5708 0" />
+    </joint>
+    <joint name="grayscale_1_joint" type="fixed">
+        <parent link="base_link" />
+        <!-- Centered, at the front, just below the chassis, facing down -->
+        <child link="grayscale_1_link" />
+        <origin xyz="${body_length/2} 0.0 ${base_link_z + 0.005}" rpy="0 1.5708 0" />
+    </joint>
+    <joint name="grayscale_2_joint" type="fixed">
+        <parent link="base_link" />
+        <!-- Slightly right, at the front, just below the chassis, facing down -->
+        <child link="grayscale_2_link" />
+        <origin xyz="${body_length/2} -0.015 ${base_link_z + 0.005}" rpy="0 1.5708 0" />
+    </joint>
 </robot>
